File: Sonda/Sonda.kicad_pcb (KiCad board)
At the start: 2 copper layers, 149.9 x 100.3 mm, 62 parts, among them J1 CONN_01X05, Q1 BC559, Q2 BC559, SW1 SW_Push, U1 ATMEGA328P-PU, U11 DS3231, U12 DataLogger, U2 MPXA6115A, U3 LM1117-3.3, U4 MPXV2010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

Commit message: PCB feito
Parts:
- moved J1 515.2 mm to (112.3, 112.8), turned to 270 degrees
- moved R2 493.5 mm to (105.4, 104.1), turned to 90 degrees
- moved D1 477.2 mm to (132.8, 84.2), turned to 180 degrees
- moved R8 476.8 mm to (101.6, 89.2), turned to 90 degrees
- moved C8 473.6 mm to (105.2, 64.0)
- moved R1 471.0 mm to (116.3, 84.2)
- moved SW1 452.9 mm to (85.7, 85.7), turned to 90 degrees
- moved JP3 447.1 mm to (104.1, 121.2), turned to 90 degrees
- moved C7 441.7 mm to (110.2, 60.5), turned to 180 degrees
- moved JP4 438.1 mm to (104.1, 126.2), turned to 90 degrees
- moved JP5 433.1 mm to (106.7, 132.1), turned to 270 degrees
- moved Q2 431.6 mm to (99.3, 59.4), turned to 90 degrees
- moved C11 429.4 mm to (81.0, 50.8), turned to 90 degrees
- moved R15 420.9 mm to (99.3, 63.2), turned to 270 degrees
- moved C4 415.6 mm to (189.0, 60.5), turned to 180 degrees
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Routing:
- net GND: track 0.00 -> 1000.0 mm, vias 0 -> 11
- net VCC: track 0.00 -> 434.4 mm, vias 0 -> 15
- net /SQW: track 0.00 -> 103.1 mm, vias 0 -> 5
- net /TX: track 0.00 -> 89.3 mm, vias 0 -> 6
- net /PD6: track 9.07 -> 93.7 mm, vias 0 -> 2
- net /SDA: track 0.00 -> 83.8 mm, vias 0 -> 4
- net /SCL: track 0.00 -> 78.0 mm, vias 0 -> 4
- net /PD7: track 8.55 -> 85.0 mm, vias 0 -> 2
- net /RX: track 0.00 -> 74.2 mm, vias 0 -> 2
- net /PC1: track 0.00 -> 72.9 mm, vias 0 -> 4
- net Net-(C11-Pad2): track 0.00 -> 66.8 mm, vias 0 -> 4
- net /RST: track 0.00 -> 65.7 mm, vias 0 -> 2
- net /ADC: track 43.4 -> 105.5 mm, vias 0 -> 6
- net Net-(C7-Pad1): track 0.00 -> 60.5 mm, vias 0 -> 6
- net Net-(BT1-Pad1): track 0.00 -> 57.7 mm
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
Commit message: PCB changes
Connections:
- U1 pad 22: Net-(U1-Pad22) -> GND
Routing:
- net GND: track 1000.0 -> 1041.5 mm, vias 11 -> 13
- net /ADC: track 105.5 -> 107.8 mm
- net /SQW: track 103.1 -> 104.1 mm, vias 5 -> 4
- net VCC: track 434.4 -> 435.1 mm, vias 15 -> 13
- net /SDA: track 83.8 -> 84.1 mm, vias 4 -> 2
- net /SCL: track 78.0 -> 78.1 mm, vias 4 -> 2
- net /PC1: vias 4 -> 2
