File: Sonda/Sonda.sch (KiCad schematic (older format))
At the start: 59 parts, among them J1 CONN_01X05, Q1 BC559, Q2 BC559, SW1 SW_Push, U1 ATMEGA328P-PU, U10 AP1117, U11 DS3231, U12 DataLogger, U2 MPXA6115A, U3 ICSP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

Commit message: modificacoes no circuito, pcb
Parts:
- removed U10: AP1117, TO_SOT_Packages_SMD:SOT-223, symbol AP1117
- removed U3: ICSP, symbol ICSP
- added C16, C17: 20pF, Capacitors_THT:C_Disc_D4.3mm_W1.9mm_P5.00mm, symbol C
- added C18: 100uF, Capacitors_THT:C_Disc_D4.3mm_W1.9mm_P5.00mm, symbol C
- added U3: LM1117-3.3, TO_SOT_Packages_THT:TO-220_Vertical, symbol LM1117-3.3
- added Y1: 16MHz, Crystals:Crystal_HC49-U_Vertical, symbol Crystal
- BT1, JP1, JP2, JP3, JP4, JP5: footprint (none) -> Pin_Headers:Pin_Header_Straight_1x02_Pitch2.54mm
- BT2: footprint (none) -> myFootprint:SuporteBateria
- C1, C10, C11, C12, C13, C15, C2, C3, C4, C5, C6, C7, C8, C9: footprint (none) -> Capacitors_THT:C_Disc_D4.3mm_W1.9mm_P5.00mm
- C14: value 0.22uF -> 10uF; footprint (none) -> Capacitors_THT:C_Disc_D4.3mm_W1.9mm_P5.00mm
- D1: footprint (none) -> LEDs:LED_D3.0mm
- J1: footprint (none) -> Pin_Headers:Pin_Header_Straight_1x05_Pitch2.54mm
- R1, R10, R11, R12, R13, R14, R15, R16, R19, R2, R20, R3, R4, R5, R6, R7, R8, R9: footprint (none) -> Resistors_THT:R_Axial_DIN0207_L6.3mm_D2.5mm_P10.16mm_Horizontal
- R17: value 2.2k -> 121; footprint (none) -> Resistors_THT:R_Axial_DIN0207_L6.3mm_D2.5mm_P10.16mm_Horizontal
- R18: value 3k -> 1k; footprint (none) -> Resistors_THT:R_Axial_DIN0207_L6.3mm_D2.5mm_P10.16mm_Horizontal
- SW1: footprint (none) -> Buttons_Switches_THT:SW_PUSH_6mm
- U1: footprint DIL28 -> Housings_DIP:DIP-28_W7.62mm_Socket_LongPads
- U11: footprint (none) -> Housings_SOIC:SOIC-16W_7.5x10.3mm_Pitch1.27mm
- U12: footprint (none) -> myFootprint:OpenLog
- U2: footprint (none) -> myFootprint:MPXH6115A
- U4, U6, U8: footprint (none) -> myFootprint:MPXV2010DP
- U5: footprint (none) -> TO_SOT_Packages_THT:TO-220_Vertical
- U7, U9: footprint (none) -> Housings_SSOP:SOP-16_4.4x10.4mm_Pitch1.27mm
Connections:
- net 3V3: now also C18.1, U3.2 (VO), U3.4 (VO)
- net GND: now also C16.1, C17.1, C18.2
- net at BT1.1 (+), C12.1, C14.1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: now also U3.3 (VI)
- net at R17.2, R18.1: now also U3.1 (GND/ADJ)
- net at U1.10 ((PCINT7/XTAL2/TOSC2)PB7): now also C17.2, Y1.2
- net at U1.9 ((PCINT6/XTAL1/TOSC1)PB6): now also C16.2, Y1.1
- no-connect marks 21 -> 16
Other:
- moved on the sheet: R17, R18

Commit message: PCB feito
Other:
- moved on the sheet: C12, C13
Changed lines of the file:
@@
 L C C12
 U 1 1 596FA1B8
-P 2300 8100
-F 0 "C12" H 2325 8200 50  0000 L CNN
-F 1 "0.33uF" H 2325 8000 50  0000 L CNN
-F 2 "Capacitors_THT:C_Disc_D4.3mm_W1.9mm_P5.00mm" H 2338 7950 50  0001 C CNN
-F 3 "" H 2300 8100 50  0001 C CNN
-	1    2300 8100
+P 2500 8100
+F 0 "C12" H 2525 8200 50  0000 L CNN
+F 1 "0.33uF" H 2525 8000 50  0000 L CNN
+F 2 "Capacitors_THT:C_Disc_D4.3mm_W1.9mm_P5.00mm" H 2538 7950 50  0001 C CNN
+F 3 "" H 2500 8100 50  0001 C CNN
+	1    2500 8100
 	1    0    0    -1
 $EndComp
@@
 L C C13
 U 1 1 596FA27B
-P 3450 8100
-F 0 "C13" H 3475 8200 50  0000 L CNN
-F 1 "0.1uF" H 3475 8000 50  0000 L CNN
-F 2 "Capacitors_THT:C_Disc_D4.3mm_W1.9mm_P5.00mm" H 3488 7950 50  0001 C CNN
-F 3 "" H 3450 8100 50  0001 C CNN
-	1    3450 8100
+P 3400 8100
+F 0 "C13" H 3425 8200 50  0000 L CNN
+F 1 "0.1uF" H 3425 8000 50  0000 L CNN
+F 2 "Capacitors_THT:C_Disc_D4.3mm_W1.9mm_P5.00mm" H 3438 7950 50  0001 C CNN
+F 3 "" H 3400 8100 50  0001 C CNN
+	1    3400 8100
 	1    0    0    -1
 $EndComp
@@
 	900  7250 900  7750
 Wire Wire Line
-	2300 7250 2300 7950
-Wire Wire Line
 	2300 7750 2550 7750
 Connection ~ 1900 7250
@@
 Wire Wire Line
 	4750 7750 5800 7750
-Connection ~ 2300 7750
 Wire Wire Line
 	2300 8250 2300 8400
 Connection ~ 2300 8400
-Wire Wire Line
-	3450 7750 3450 7950
-Connection ~ 3450 7750
 Wire Wire Line
 	3450 8250 3450 8400
@@
 	5400 8750 5400 8350
 Connection ~ 5050 8750
+Wire Wire Line
+	2300 7250 2300 7750
+Wire Wire Line
+	2500 7950 2500 7750
+Connection ~ 2500 7750
+Wire Wire Line
+	2300 8250 2500 8250
+Wire Wire Line
+	3450 8250 3400 8250
+Wire Wire Line
+	3400 7950 3400 7750
+Connection ~ 3400 7750
 $EndSCHEMATC

Commit message: PCB changes
Connections:
- net GND: now also U1.22 (GND)
- no-connect marks 16 -> 15
Changed lines of the file:
@@
 NoConn ~ 1100 1300
 NoConn ~ 1100 1600
-NoConn ~ 1100 3200
 NoConn ~ 3000 1000
 NoConn ~ 3000 1100
@@
 	3400 7950 3400 7750
 Connection ~ 3400 7750
+Wire Wire Line
+	1100 3200 900  3200
+Text Label 900  3200 0    60   ~ 0
+GND
 $EndSCHEMATC
